File: keyboard.kicad_sch (KiCad schematic)
At the start: 2 parts, among them SW1 SW_Push, SW2 SW_Push

Commit message: ファイル追加
Parts:
- removed SW2: SW_Push, kbd_SW:CherryMX_Solder_1.25u, symbol Switch:SW_Push
- added D: D, symbol Device:D
- added D0-0, D0-1, D0-10, D0-11, D0-12, D0-13, D0-14, D0-15, D0-2, D0-3, D0-4, D0-5, D0-6, D0-7, D0-8, D0-9, D1-0, D1-1, D1-10, D1-11, D1-12, D1-13, D1-14, D1-15, D1-16, D1-17, D1-18, D1-19, D1-2, D1-20, D1-3, D1-4, D1-5, D1-6, D1-7, D1-8, D1-9, D2-0, D2-1, D2-10, D2-11, D2-12, D2-13, D2-14, D2-15, D2-16, D2-17, D2-18, D2-19, D2-2, D2-20, D2-3, D2-4, D2-5, D2-6, D2-7, D2-8, D2-9, D3-0, D3-1, D3-10, D3-11, D3-12, D3-13, D3-14, D3-15, D3-2, D3-3, D3-4, D3-5, D3-6, D3-7, D3-8, D3-9, D4-0, D4-1, D4-10, D4-11, D4-12, D4-13, D4-14, D4-15, D4-16, D4-17, D4-2, D4-3, D4-4, D4-5, D4-6, D4-7, D4-8, D4-9, D5-0, D5-1, D5-10, D5-11, D5-12, D5-2, D5-3, D5-4, D5-5, D5-6, D5-7, D5-8, D5-9: D, kbd_Parts:Diode_SMD, symbol Device:D
- added SW0-0, SW0-1, SW0-10, SW0-11, SW0-12, SW0-13, SW0-14, SW0-15, SW0-2, SW0-3, SW0-4, SW0-5, SW0-6, SW0-7, SW0-8, SW0-9, SW1-0, SW1-1, SW1-10, SW1-11, SW1-12, SW1-13, SW1-14, SW1-15, SW1-16, SW1-17, SW1-18, SW1-19, SW1-2, SW1-20, SW1-3, SW1-4, SW1-5, SW1-6, SW1-7, SW1-8, SW1-9, SW2-0, SW2-1, SW2-10, SW2-11, SW2-12, SW2-13, SW2-14, SW2-15, SW2-16, SW2-17, SW2-18, SW2-19, SW2-2, SW2-20, SW2-3, SW2-4, SW2-5, SW2-6, SW2-7, SW2-8, SW2-9, SW3-0, SW3-1, SW3-10, SW3-11, SW3-12, SW3-13, SW3-14, SW3-15, SW3-2, SW3-3, SW3-4, SW3-5, SW3-6, SW3-7, SW3-8, SW3-9, SW4-0, SW4-1, SW4-10, SW4-11, SW4-12, SW4-13, SW4-14, SW4-15, SW4-16, SW4-17, SW4-2, SW4-3, SW4-4, SW4-5, SW4-6, SW4-7, SW4-8, SW4-9, SW5-0, SW5-1, SW5-10, SW5-11, SW5-12, SW5-2, SW5-3, SW5-4, SW5-5, SW5-6, SW5-7, SW5-8, SW5-9: SW_Push, kbd_SW:CherryMX_Solder_1u, symbol Switch:SW_Push
- renumbered SW1 to SW
Connections:
- new net: D2-2.2 (A), SW2-2.2
- new net: D5-10.2 (A), SW5-10.2
- new net: D1-3.2 (A), SW1-3.2
- new net: D4-15.2 (A), SW4-15.2
- new net: D4-6.2 (A), SW4-6.2
- new net: D1-13.2 (A), SW1-13.2
- new net: D3-0.2 (A), SW3-0.2
- new net: D0-14.2 (A), SW0-14.2
- new net: D1-14.2 (A), SW1-14.2
- new net: D5-4.2 (A), SW5-4.2
- new net: D5-7.2 (A), SW5-7.2
- new net: D2-20.2 (A), SW2-20.2
- new net: D1-15.2 (A), SW1-15.2
- new net: D3-10.2 (A), SW3-10.2
- new net: D4-4.2 (A), SW4-4.2
- new net: D1-2.2 (A), SW1-2.2
- new net: D1-0.2 (A), SW1-0.2
- new net: D4-13.2 (A), SW4-13.2
- new net: D1-4.2 (A), SW1-4.2
- new net: D2-19.2 (A), SW2-19.2
- new net: D2-6.2 (A), SW2-6.2
- new net: D1-12.2 (A), SW1-12.2
- new net: D4-16.2 (A), SW4-16.2
- new net: D3-2.2 (A), SW3-2.2
- new net: D5-12.2 (A), SW5-12.2
- new net: D2-18.2 (A), SW2-18.2
- new net: D0-0.2 (A), SW0-0.2
- new net: D4-1.2 (A), SW4-1.2
- new net: D5-6.2 (A), SW5-6.2
- new net: D1-18.2 (A), SW1-18.2
- new net: D4-12.2 (A), SW4-12.2
- new net: D0-1.2 (A), SW0-1.2
- new net: D3-12.2 (A), SW3-12.2
- new net: D2-12.2 (A), SW2-12.2
- new net: D4-7.2 (A), SW4-7.2
- new net: D2-10.2 (A), SW2-10.2
- new net: D0-12.2 (A), SW0-12.2
- new net: D4-11.2 (A), SW4-11.2
- new net: D1-19.2 (A), SW1-19.2
- new net: D0-7.2 (A), SW0-7.2
- new net: D2-7.2 (A), SW2-7.2
- new net: D5-2.2 (A), SW5-2.2
- new net: D0-4.2 (A), SW0-4.2
- new net: D1-17.2 (A), SW1-17.2
- new net: D1-5.2 (A), SW1-5.2
- new net: D3-5.2 (A), SW3-5.2
- new net: D4-14.2 (A), SW4-14.2
- new net: D5-5.2 (A), SW5-5.2
- new net: D0-9.2 (A), SW0-9.2
- new net: D0-2.2 (A), SW0-2.2
- new net: D5-1.2 (A), SW5-1.2
- new net: D1-11.2 (A), SW1-11.2
- new net: D2-13.2 (A), SW2-13.2
- new net: D4-0.2 (A), SW4-0.2
- new net: D2-1.2 (A), SW2-1.2
- new net: D5-3.2 (A), SW5-3.2
- new net: D3-1.2 (A), SW3-1.2
- new net: D1-16.2 (A), SW1-16.2
- new net: D0-8.2 (A), SW0-8.2
- new net: D5-8.2 (A), SW5-8.2
- new net: D1-7.2 (A), SW1-7.2
- new net: D3-9.2 (A), SW3-9.2
- new net: D4-5.2 (A), SW4-5.2
- new net: D0-6.2 (A), SW0-6.2
- new net: D0-15.2 (A), SW0-15.2
- new net: D3-8.2 (A), SW3-8.2
- new net: D3-3.2 (A), SW3-3.2
- new net: D2-0.2 (A), SW2-0.2
- new net: D3-13.2 (A), SW3-13.2
- new net: D2-11.2 (A), SW2-11.2
- new net: D2-9.2 (A), SW2-9.2
- new net: D4-9.2 (A), SW4-9.2
- new net: D2-16.2 (A), SW2-16.2
- new net: D2-5.2 (A), SW2-5.2
- new net: D1-9.2 (A), SW1-9.2
- new net: D0-5.2 (A), SW0-5.2
- new net: D2-3.2 (A), SW2-3.2
- new net: D1-1.2 (A), SW1-1.2
- new net: D1-6.2 (A), SW1-6.2
- new net: D4-2.2 (A), SW4-2.2
- new net: D1-20.2 (A), SW1-20.2
- new net: D0-11.2 (A), SW0-11.2
- new net: D2-14.2 (A), SW2-14.2
- new net: D2-8.2 (A), SW2-8.2
- new net: D1-10.2 (A), SW1-10.2
- new net: D3-15.2 (A), SW3-15.2
- new net: D0-3.2 (A), SW0-3.2
- new net: D3-4.2 (A), SW3-4.2
- new net: D2-4.2 (A), SW2-4.2
- new net: D5-0.2 (A), SW5-0.2
- new net: D3-7.2 (A), SW3-7.2
- new net: D3-6.2 (A), SW3-6.2
- new net: D0-13.2 (A), SW0-13.2
- new net: D3-14.2 (A), SW3-14.2
- new net: D4-8.2 (A), SW4-8.2
- new net: D2-15.2 (A), SW2-15.2
- new net: D4-3.2 (A), SW4-3.2
- new net: D2-17.2 (A), SW2-17.2
- new net: D3-11.2 (A), SW3-11.2
- new net: D5-9.2 (A), SW5-9.2
- new net: D5-11.2 (A), SW5-11.2
- new net: D4-17.2 (A), SW4-17.2
- new net: D4-10.2 (A), SW4-10.2
- new net: D0-10.2 (A), SW0-10.2
- new net: D1-8.2 (A), SW1-8.2
- new net COL0: SW0-0.1, SW1-0.1, SW2-0.1, SW3-0.1, SW4-0.1, SW5-0.1
- new net COL1: SW0-1.1, SW1-1.1, SW2-1.1, SW3-1.1, SW4-1.1, SW5-1.1
- new net COL10: SW0-10.1, SW1-10.1, SW2-10.1, SW3-10.1, SW4-10.1, SW5-10.1
- new net COL11: SW0-11.1, SW1-11.1, SW2-11.1, SW3-11.1, SW4-11.1, SW5-11.1
- new net COL12: SW0-12.1, SW1-12.1, SW2-12.1, SW3-12.1, SW4-12.1, SW5-12.1
- new net COL13: SW0-13.1, SW1-13.1, SW2-13.1, SW3-13.1, SW4-13.1
- new net COL14: SW0-14.1, SW1-14.1, SW2-14.1, SW3-14.1, SW4-14.1
- new net COL15: SW0-15.1, SW1-15.1, SW2-15.1, SW3-15.1, SW4-15.1
- new net COL16: SW1-16.1, SW2-16.1, SW4-16.1
- new net COL17: SW1-17.1, SW2-17.1, SW4-17.1
- new net COL18: SW1-18.1, SW2-18.1
- new net COL19: SW1-19.1, SW2-19.1
- new net COL2: SW0-2.1, SW1-2.1, SW2-2.1, SW3-2.1, SW4-2.1, SW5-2.1
- new net COL20: SW1-20.1, SW2-20.1
- new net COL3: SW0-3.1, SW1-3.1, SW2-3.1, SW3-3.1, SW4-3.1, SW5-3.1
- new net COL4: SW0-4.1, SW1-4.1, SW2-4.1, SW3-4.1, SW4-4.1, SW5-4.1
- new net COL5: SW0-5.1, SW1-5.1, SW2-5.1, SW3-5.1, SW4-5.1, SW5-5.1
- new net COL6: SW0-6.1, SW1-6.1, SW2-6.1, SW3-6.1, SW4-6.1, SW5-6.1
- new net COL7: SW0-7.1, SW1-7.1, SW2-7.1, SW3-7.1, SW4-7.1, SW5-7.1
- new net COL8: SW0-8.1, SW1-8.1, SW2-8.1, SW3-8.1, SW4-8.1, SW5-8.1
- new net COL9: SW0-9.1, SW1-9.1, SW2-9.1, SW3-9.1, SW4-9.1, SW5-9.1
- new net ROW0: D0-0.1 (K), D0-1.1 (K), D0-10.1 (K), D0-11.1 (K), D0-12.1 (K), D0-13.1 (K), D0-14.1 (K), D0-15.1 (K), D0-2.1 (K), D0-3.1 (K), D0-4.1 (K), D0-5.1 (K), D0-6.1 (K), D0-7.1 (K), D0-8.1 (K), D0-9.1 (K)
- new net ROW1: D1-0.1 (K), D1-1.1 (K), D1-10.1 (K), D1-11.1 (K), D1-12.1 (K), D1-13.1 (K), D1-14.1 (K), D1-15.1 (K), D1-16.1 (K), D1-17.1 (K), D1-18.1 (K), D1-19.1 (K), D1-2.1 (K), D1-20.1 (K), D1-3.1 (K), D1-4.1 (K), D1-5.1 (K), D1-6.1 (K), D1-7.1 (K), D1-8.1 (K), D1-9.1 (K)
- new net ROW2: D2-0.1 (K), D2-1.1 (K), D2-10.1 (K), D2-11.1 (K), D2-12.1 (K), D2-13.1 (K), D2-14.1 (K), D2-15.1 (K), D2-16.1 (K), D2-17.1 (K), D2-18.1 (K), D2-19.1 (K), D2-2.1 (K), D2-20.1 (K), D2-3.1 (K), D2-4.1 (K), D2-5.1 (K), D2-6.1 (K), D2-7.1 (K), D2-8.1 (K), D2-9.1 (K)
- new net ROW3: D3-0.1 (K), D3-1.1 (K), D3-10.1 (K), D3-11.1 (K), D3-12.1 (K), D3-13.1 (K), D3-14.1 (K), D3-15.1 (K), D3-2.1 (K), D3-3.1 (K), D3-4.1 (K), D3-5.1 (K), D3-6.1 (K), D3-7.1 (K), D3-8.1 (K), D3-9.1 (K)
- new net ROW4: D4-0.1 (K), D4-1.1 (K), D4-10.1 (K), D4-11.1 (K), D4-12.1 (K), D4-13.1 (K), D4-14.1 (K), D4-15.1 (K), D4-16.1 (K), D4-17.1 (K), D4-2.1 (K), D4-3.1 (K), D4-4.1 (K), D4-5.1 (K), D4-6.1 (K), D4-7.1 (K), D4-8.1 (K), D4-9.1 (K)
- new net ROW5: D5-0.1 (K), D5-1.1 (K), D5-10.1 (K), D5-11.1 (K), D5-12.1 (K), D5-2.1 (K), D5-3.1 (K), D5-4.1 (K), D5-5.1 (K), D5-6.1 (K), D5-7.1 (K), D5-8.1 (K), D5-9.1 (K)
Other:
- moved on the sheet: SW
